File: pcb/DIR.kicad_sch (KiCad schematic)
At the start: 58 parts, among them J1 USB_C_Receptacle, J2 Conn_01x02_Pin, Q1 BSP613, SW1 SW_SPDT, U1 MCP73833, U2 TPS61023DRLR

Commit message: Fix wrong vendor-id
Parts:
- D2: VendorId 100188 -> 100194
Changed lines of the file:
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@@
       (effects (font (size 1.27 1.27)) hide)
     )
-    (property "VendorId" "100188" (at 265.43 69.85 0)
+    (property "VendorId" "100194" (at 265.43 69.85 0)
       (effects (font (size 1.27 1.27)) hide)
     )

Commit message: Change Z-Diode to 3V3
Parts:
- D2: value BZV55B5V6 -> BZV33B3V3; VendorId 100194 -> 100187
Changed lines of the file:
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@@
       (effects (font (size 1.27 1.27)) (justify left))
     )
-    (property "Value" "BZV55B5V6" (at 267.97 69.85 0)
+    (property "Value" "BZV33B3V3" (at 267.97 69.85 0)
       (effects (font (size 1.27 1.27)))
     )
@@
       (effects (font (size 1.27 1.27)) hide)
     )
-    (property "VendorId" "100194" (at 265.43 69.85 0)
+    (property "VendorId" "100187" (at 265.43 69.85 0)
       (effects (font (size 1.27 1.27)) hide)
     )

Commit message: Fix power path issue
Parts:
- removed C8: 100n, Capacitor_SMD:C_1206_3216Metric, symbol Device:C
- added C8: 10u, Capacitor_Tantalum_SMD:CP_EIA-6032-28_Kemet-C, symbol Device:C_Polarized
- added U8: LM1117DT-3.3, Package_TO_SOT_SMD:TO-252-3_TabPin2, symbol Regulator_Linear:LM1117DT-3.3
- D2: value BZV33B3V3 -> BZV36B3V6; VendorId 100187 -> 100189
- R3: value 680k -> 732k; VendorId 102997 -> 193602
- R8: value 150k -> 100k; VendorId 102989 -> 102987
Connections:
- net +3V3: now also U8.2 (VO); no longer C15.1, C16.1, C17.1, C18.1, C19.1, C20.1, C7.1, R3.2, TP4.1, U2.6 (VOUT)
- net +5V: now also C15.1, C16.1, C17.1, C18.1, C19.1, C20.1, C7.1, R3.2, TP4.1, U2.6 (VOUT), C8.1, U8.3 (VI)
- net GND: now also C8.2, U8.1 (GND)
Other:
- moved on the sheet: C1, C10, C11, C12, C13, C14, C15, C16, C17, C18, C19, C2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
